Commit message: fixed some problem

File: catkin_ws/src/senior_akm_robot/xacro/senior_akm.xacro (robot description, xacro)
@@ -1,21 +1,21 @@
 <?xml version="1.0"?>
 <robot name="wheeltec" xmlns:xacro="http://www.ros.org/wiki/xacro">
-    <!--M_PI-->
+    <!-- M_PI-->
     <xacro:property name="M_PI" value="3.1415926535897931" />
-    <!--rplidar description-->
-    <!--rplidar position-->
-    <xacro:property name="rplidar_position_x" value="0.0887405189187401" />
+    <!-- rplidar description-->
+    <!-- rplidar position-->
+    <xacro:property name="rplidar_position_x" value="0.0887" />
     <xacro:property name="rplidar_position_y" value="0.000667202411597726" />
     <xacro:property name="rplidar_position_z" value="0.111024183741431" />
-    <!--rplidar scanning angle-->
-    <xacro:property name="rplidar_min_angle" value="-120" />
-    <xacro:property name="rplidar_max_angle" value="120" />
-    <!--camera description-->
-    <!--camera position-->
+    <!-- rplidar scanning angle-->
+    <xacro:property name="rplidar_min_angle" value="-150" />
+    <xacro:property name="rplidar_max_angle" value="150" />
+    <!-- camera description-->
+    <!-- camera position-->
     <xacro:property name="camera_position_x" value="0.165778518918356" />
     <xacro:property name="camera_position_y" value="0.000945202408300414" />
     <xacro:property name="camera_position_z" value="0.089704" />
-    <!--robot_body description-->
-    <!--wheel position-->
+    <!-- robot_body description-->
+    <!-- wheel position-->
     <xacro:property name="rear_wheel_position_x" value="-0.157526481081644" />
     <xacro:property name="right_rear_wheel_position_y" value="-0.154348797591698" />
@@ -27,17 +27,17 @@
     <xacro:property name="right_front_wheel_position_y" value="-0.1529487975917" />
     <xacro:property name="front_wheel_position_z" value="0.0241" />
-    <xacro:property name="wheel_mass" value="0.4"/>
-    <!--chassis position-->
+    <xacro:property name="wheel_mass" value="0.4" />
+    <!-- chassis position-->
     <xacro:property name="box_position_x" value="-0.056" />
     <xacro:property name="box_position_y" value="0" />
     <xacro:property name="box_position_z" value="0.0632418734279548" />
-    <!--chassis inertia-->
+    <!-- chassis inertia-->
     <xacro:property name="box_length" value="0.445" />
     <xacro:property name="box_height" value="0.206" />
     <xacro:property name="box_width" value="0.36" />
-    <xacro:property name="box_mass" value="8" />
-    <!--wheel angle limit-->
-    <xacro:property name="wheel_travel" value="1.046562"/> <!--60 degree-->
-    <!--robot with rplidar,camera and imu -->
+    <xacro:property name="box_mass" value="10" />
+    <!-- wheel angle limit-->
+    <xacro:property name="wheel_travel" value="0.69813" /> <!-- 40 degree-->
+    <!-- robot with rplidar,camera and imu -->
     <xacro:include filename="$(find senior_akm_robot)/xacro/senior_akm_body.xacro" />
     <xacro:include filename="$(find senior_akm_robot)/xacro/senior_akm_rplidar.xacro" />
@@ -46,122 +46,123 @@
     <xacro:include filename="$(find senior_akm_robot)/xacro/material.xacro" />
     <xacro:include filename="$(find senior_akm_robot)/xacro/senior_akm_transmission.xacro" />
+    <xacro:include filename="$(find senior_akm_robot)/xacro/contact.xacro" />
     <!-- define rplidar joint-->
     <joint name="rplidar_joint" type="fixed">
         <origin xyz="${rplidar_position_x} ${rplidar_position_y} ${rplidar_position_z}" rpy="0 0 0" />
-        <parent link="base_link"/>
-        <child link="laser_link"/>
+        <parent link="base_link" />
+        <child link="laser_link" />
     </joint>
     <!-- define camera joint-->
     <joint name="camera_frame_joint" type="fixed">
         <origin xyz="${camera_position_x} ${camera_position_y} ${camera_position_z}" rpy="0 0 0" />
-        <parent link="base_link"/>
-        <child link="camera_link"/>
+        <parent link="base_link" />
+        <child link="camera_link" />
     </joint>
-    <!--define rear_wheel_joint rotate around the y axis,Max velocity is 38.70 rad/s,Max effort 3.9 N m  -->
+    <!-- define rear_wheel_joint rotate around the y axis,Max velocity is 38.70 rad/s,Max effort 3.9 N m  -->
     <xacro:macro name="rear_joint" params="LR *origin  ">
-    <joint name="${LR}_rear_wheel_joint" type="continuous">
-        <xacro:insert_block name="origin"/>
-        <parent link="base_link"/>
-        <child link="${LR}_rear_wheel_link"/>
-        <axis xyz="0 1 0" rpy="0 0 0"/>
-        <limit effort="3.9" velocity="38.70"/>
-    </joint>
+        <joint name="${LR}_rear_wheel_joint" type="continuous">
+            <xacro:insert_block name="origin" />
+            <parent link="base_link" />
+            <child link="${LR}_rear_wheel_link" />
+            <axis xyz="0 1 0" rpy="0 0 0" />
+            <limit effort="1.0" velocity="38.70" />
+        </joint>
     </xacro:macro>
     <xacro:macro name="front_joint" params="LR *origin ">
-        <!--define front axle carrier-->
-    <link name="${LR}_front_axle_carrier">
-        <inertial>
-          <mass value="0.01"/>
-          <inertia ixx="0.001" ixy="0" ixz="0" iyy="0.001" iyz="0" izz="0.001"/>
-        </inertial>
-    </link>
-        <!--define front_wheel_joint rotate around the y axis,Max velocity is 38.70 rad/s,Max effort 3.9 N m-->
-    <joint name="${LR}_front_wheel_joint" type="continuous">
-        <origin xyz="0 0 0" rpy="0 0 0"/>
-        <parent link="${LR}_front_axle_carrier"/>
-        <child link="${LR}_front_wheel_link"/>
-        <axis xyz="0 1 0" rpy="0 0 0"/>
-        <limit effort="3.9" velocity="38.70" />
+        <!-- define front axle carrier-->
+        <link name="${LR}_front_axle_carrier">
+            <inertial>
+                <mass value="0.01" />
+                <inertia ixx="0.001" ixy="0" ixz="0" iyy="0.001" iyz="0" izz="0.001" />
+            </inertial>
+        </link>
+        <!-- define front_wheel_joint rotate around the y axis,Max velocity is 38.70 rad/s,Max effort 3.9 N m-->
+        <joint name="${LR}_front_wheel_joint" type="continuous">
+            <origin xyz="0 0 0" rpy="0 0 0" />
+            <parent link="${LR}_front_axle_carrier" />
+            <child link="${LR}_front_wheel_link" />
+            <axis xyz="0 1 0" rpy="0 0 0" />
+            <limit effort="1.0" velocity="38.70" />
+        </joint>
+        <!-- define steering_joint rotate around the z axis,Max velocity is 4.5 rad/s,Max effort 0.045 N m-->
+        <joint name="${LR}_steering_joint" type="revolute">
+            <xacro:insert_block name="origin" />
+            <parent link="base_link" />
+            <child link="${LR}_front_axle_carrier" />
+            <axis xyz="0 0 1" />
+            <!-- upper 30 degree and lower -30 degree-->
+            <limit lower="${-wheel_travel/2}" upper="${wheel_travel/2}"
+                effort="0.045" velocity="4.5" />
+        </joint>
+    </xacro:macro>
+    <!-- define imu_joint fixed -->
+    <joint name="imu_joint" type="fixed">
+        <origin xyz="-0.03 0 0.06" rpy="0 0 0" />
+        <parent link="base_link" />
+        <child link="imu_link" />
     </joint>
-        <!--define steering_joint rotate around the z axis,Max velocity is 4.5 rad/s,Max effort 0.045 N m-->
-    <joint name="${LR}_steering_joint" type="revolute">
-      <xacro:insert_block name="origin"/>
-      <parent link="base_link"/>
-      <child link="${LR}_front_axle_carrier"/>
-      <axis xyz="0 0 1"/>
-            <!--upper 30 degree and lower -30 degree-->
-      <limit lower="${-wheel_travel/2}" upper="${wheel_travel/2}"
-             effort="0.045" velocity="4.5"/>
-    </joint>
-    </xacro:macro>
-    <!--define imu_joint fixed -->
-    <joint name="imu_joint" type="fixed">
-      <origin xyz="-0.03 0 0.06" rpy="0 0 0" />
-      <parent link="base_link"/>
-      <child link="imu_link"/>
-    </joint>
-    <!--macro call rplidar imu astra_camera-->
-    <rplidar LA="laser"/>
-    <imu prefix="imu"/>
-    <astra_camera prefix="camera"/>
-    <!--macro call wheel_link-->
+    <!-- macro call rplidar imu astra_camera-->
+    <rplidar LA="laser" />
+    <imu prefix="imu" />
+    <astra_camera prefix="camera" />
+    <!-- macro call wheel_link-->
     <xacro:wheel_link LR="right" FR="rear">
         <origin xyz="-3.98258093170512E-11 -0.00279452473049574 1.19940203602287E-11" rpy="0 0 0" />
         <inertia
-          ixx="1.99603833653634E-05"
-          ixy="1.47023522649957E-14"
-          ixz="1.56178238251791E-10"
-          iyy="3.41116766443603E-05"
-          iyz="-1.59750652595274E-15"
-          izz="1.99606952584451E-05" />
+            ixx="1.99603833653634E-05"
+            ixy="1.47023522649957E-14"
+            ixz="1.56178238251791E-10"
+            iyy="3.41116766443603E-05"
+            iyz="-1.59750652595274E-15"
+            izz="1.99606952584451E-05" />
     </xacro:wheel_link>
     <xacro:wheel_link LR="left" FR="rear">
         <origin xyz="3.98258093170512E-11 0.00279452473049574 1.19940203602287E-11" rpy="0 0 0" />
         <inertia
-          ixx="1.99603833653634E-05"
-          ixy="1.47023522649957E-14"
-          ixz="-1.56178238251791E-10"
-          iyy="3.41116766443603E-05"
-          iyz="1.59750652595274E-15"
-          izz="1.99606952584451E-05" />
+            ixx="1.99603833653634E-05"
+            ixy="1.47023522649957E-14"
+            ixz="-1.56178238251791E-10"
+            iyy="3.41116766443603E-05"
+            iyz="1.59750652595274E-15"
+            izz="1.99606952584451E-05" />
     </xacro:wheel_link>
     <xacro:wheel_link LR="right" FR="front">
         <origin xyz="1.50883194827145E-11 -0.00228176069832715 1.40150807625972E-11" rpy="0 0 0" />
         <inertia
-          ixx="1.91351003010526E-05"
-          ixy="-4.51400783455223E-15"
-          ixz="-2.66123995114195E-10"
-          iyy="3.30131998434901E-05"
-          iyz="-4.48462029754282E-15"
-          izz="1.91374249680472E-05" />
+            ixx="1.91351003010526E-05"
+            ixy="-4.51400783455223E-15"
+            ixz="-2.66123995114195E-10"
+            iyy="3.30131998434901E-05"
+            iyz="-4.48462029754282E-15"
+            izz="1.91374249680472E-05" />
     </xacro:wheel_link>
     <xacro:wheel_link LR="left" FR="front">
-        <origin xyz="1.50882639715633E-11 0.00228176069832718 -1.40150807625972E-11" rpy="0 0 0"  />
+        <origin xyz="1.50882639715633E-11 0.00228176069832718 -1.40150807625972E-11" rpy="0 0 0" />
         <inertia
-          ixx="1.91343292762451E-05"
-          ixy="4.51397364480803E-15"
-          ixz="9.52734291190626E-10"
-          iyy="3.30122388976539E-05"
-          iyz="-4.48462116122782E-15"
-          izz="1.91372350470185E-05" />
+            ixx="1.91343292762451E-05"
+            ixy="4.51397364480803E-15"
+            ixz="9.52734291190626E-10"
+            iyy="3.30122388976539E-05"
+            iyz="-4.48462116122782E-15"
+            izz="1.91372350470185E-05" />
     </xacro:wheel_link>
-    <!--macro call rear_joint-->
-    <xacro:rear_joint LR="right" >
+    <!-- macro call rear_joint-->
+    <xacro:rear_joint LR="right">
         <origin xyz="${rear_wheel_position_x} ${right_rear_wheel_position_y} ${rear_wheel_position_z}" rpy="0 0 0" />
     </xacro:rear_joint>
-    <xacro:rear_joint LR="left" >
+    <xacro:rear_joint LR="left">
         <origin xyz="${rear_wheel_position_x} ${left_rear_wheel_position_y} ${rear_wheel_position_z}" rpy="0 0 0" />
     </xacro:rear_joint>
-    <xacro:front_joint LR="right" >
+    <xacro:front_joint LR="right">
         <origin xyz="${right_front_wheel_position_x} ${right_front_wheel_position_y} ${front_wheel_position_z}" rpy="0 0 0" />
     </xacro:front_joint>
-    <xacro:front_joint LR="left" >
+    <xacro:front_joint LR="left">
         <origin xyz="${left_front_wheel_position_x} ${left_front_wheel_position_y} ${front_wheel_position_z}" rpy="0 0 0" />
     </xacro:front_joint>
-    <!--macro call transmission-->
-    <wheel_transmission LR="right" FR="rear"/>
-    <wheel_transmission LR="left" FR="rear"/>
-    <wheel_transmission LR="right" FR="front"/>
-    <wheel_transmission LR="left" FR="front"/>
+    <!-- macro call transmission-->
+    <wheel_transmission LR="right" FR="rear" />
+    <wheel_transmission LR="left" FR="rear" />
+    <wheel_transmission LR="right" FR="front" />
+    <wheel_transmission LR="left" FR="front" />
     <steering_transmission LR="right" />
     <steering_transmission LR="left" />

File: catkin_ws/src/senior_akm_robot/xacro/senior_akm_body.xacro (robot description, xacro)
@@ -23,5 +23,5 @@
     </xacro:macro>
     <!-- define base_footprint -->
-    <link name="base_footprint" />
+    <link name="base_footprint"></link>
     <!-- define fixed base_footprint_joint -->
     <joint

File: catkin_ws/src/senior_akm_robot/xacro/senior_akm_rplidar.xacro (robot description, xacro)
@@ -30,11 +30,11 @@
             sensor-->
             <sensor type="ray" name="rplidar">
-                <visualize>false</visualize>
+                <visualize>true</visualize>
                 <update_rate>12</update_rate>
                 <ray>
                     <scan>
                         <horizontal>
-                            <samples>600</samples>
-                            <resolution>0.4</resolution>
+                            <samples>750</samples>
+                            <!-- <resolution>0.4</resolution> -->
                             <min_angle>${rplidar_min_angle*M_PI/180}</min_angle>
                             <max_angle>${rplidar_max_angle*M_PI/180}</max_angle>
@@ -46,6 +46,5 @@
                         <resolution>0.01</resolution>
                     </range>
-                    <!--Add
-                    gaussian noise-->
+                    <!-- Add gaussian noise-->
                     <noise>
                         <type>gaussian</type>

File: catkin_ws/src/senior_akm_robot/xacro/senior_akm_transmission.xacro (robot description, xacro)
@@ -21,8 +21,8 @@
             <type>transmission_interface/SimpleTransmission</type>
             <joint name="${LR}_${FR}_wheel_joint">
-                <hardwareInterface>VelocityJointInterface</hardwareInterface>
+                <hardwareInterface>hardware_interface/VelocityJointInterface</hardwareInterface>
             </joint>
             <actuator name="${LR}_${FR}_wheel_joint_motor">
-                <hardwareInterface>VelocityJointInterface</hardwareInterface>
+                <hardwareInterface>hardware_interface/VelocityJointInterface</hardwareInterface>
                 <mechanicalReduction>1</mechanicalReduction>
             </actuator>
@@ -33,8 +33,8 @@
             <type>transmission_interface/SimpleTransmission</type>
             <joint name="${LR}_steering_joint">
-                <hardwareInterface>PositionJointInterface</hardwareInterface>
+                <hardwareInterface>hardware_interface/PositionJointInterface</hardwareInterface>
             </joint>
             <actuator name="${LR}_steering_act">
-                <hardwareInterface>PositionJointInterface</hardwareInterface>
+                <hardwareInterface>hardware_interface/PositionJointInterface</hardwareInterface>
                 <mechanicalReduction>1</mechanicalReduction>
             </actuator>

Commit message: add:a good model

File: catkin_ws/src/senior_akm_robot/xacro/senior_akm.xacro (robot description, xacro)
@@ -66,5 +66,5 @@
             <child link="${LR}_rear_wheel_link" />
             <axis xyz="0 1 0" rpy="0 0 0" />
-            <limit effort="1.0" velocity="38.70" />
+            <limit effort="1.0" velocity="28.70" />
         </joint>
     </xacro:macro>
@@ -83,5 +83,5 @@
             <child link="${LR}_front_wheel_link" />
             <axis xyz="0 1 0" rpy="0 0 0" />
-            <limit effort="1.0" velocity="38.70" />
+            <limit effort="1.0" velocity="28.70" />
         </joint>
         <!-- define steering_joint rotate around the z axis,Max velocity is 4.5 rad/s,Max effort 0.045 N m-->
