Commit message: add: new map

File: catkin_ws/src/senior_akm_robot/urdf/senior_akm.urdf (robot description, URDF)
Before this commit: robot wheeltec, 12 links, 11 joints
Joints:
- joint rplidar_joint: origin xyz=0.0887405189187 0.000667202411598 0.111024183741 rpy=0 0 0 -> xyz=0 0.000667202411598 0.111024183741 rpy=0 0 0
